Commit message: feat(nav2): Step 4·5 — 파라미터 확정 + Nav2 기동 launch (장소 프리셋)
시뮬에서 목표를 찍으면 자율주행이 되는 지점까지 완성.

■ 설정 구조 — "공통 1 + 장소별 1"
  시연 당일 YAML을 여는 것은 사고가 나고, 설정 전체를 두 벌 복사하면
  한쪽만 고치고 다른 쪽을 잊는다. 공통은 한 곳에 두고 다른 값 4개만 분리.
  명령어의 space 단어 하나가 4가지를 동시에 바꾼다.

      항목                    narrow   wide     파일
      local_costmap 크기      2x2      5x5      space_*.yaml
      local/global inflation  0.10     0.25     space_*.yaml
      복구 행동 spin          미사용   사용     navigate_*.xml

  ROS 2는 --params-file을 여러 개 받으면 나중 파일이 이긴다. overlay에
  적은 값만 덮어써지고 나머지는 공통 파일 값이 유지되는 것을 실측 확인.

■ 값의 근거
  속도 0.15 m/s, 0.6 rad/s — 슬램 담당자 설정을 그대로 따름
  가속 = 속도 / 최고속 도달시간 0.5초 → 0.30 m/s², 1.20 rad/s²
  JGB37-520 사양표로 상한 확인: 채택값이 모터 한계의 4.9%,
  바퀴 슬립 한계(4.61 m/s²)의 6.5%. 실물 실측이 불필요함을 확정.

■ cmd_vel 은 velocity_smoother 를 반드시 거친다
      controller --(/cmd_vel_nav)--> smoother --(/cmd_vel)--> 로봇
  Nav2 기본은 controller가 /cmd_vel을 직접 쏘는데, 그러면 가속 제한이
  적용되지 않는다. 실물 펌웨어에도 wheel_odom_bridge에도 클램프가 없어
  속도·가속을 제한할 수 있는 곳이 여기뿐이다.

■ 작업 중 잡은 문제
  - plugin_lib_names를 줄였다가 Nav2 전체가 안 뜸. bt_navigator는 트리를
    두 개 로드하므로 Humble 기준 47개 전체가 필요 (RemovePassedGoals 누락)
  - use_cost_regulated_linear_velocity_scaling: 작은 방에서 팽창 영역이
    바닥 전체를 덮어 상시 감속. 끄니 평균 0.050 → 0.116~0.130 m/s
  - behavior_server가 최신 Nav2 문법이었음. Humble은 costmap_topic 단수형
    이고 global_frame은 map이 아니라 odom. 선언 안 된 파라미터는 경고도
    없이 무시되므로 Humble 기준 파일과 직접 대조해서 발견
  - RViz 노란 선: /local_plan은 DWB 전용. RPP는 lookahead_collision_arc
  - 전방주시를 늘렸다가 되돌림. 추종점이 차체 안에 찍히는 것은 차동구동
    에서는 문제가 아니다(제어점이 base_link, 제자리 회전 가능)

■ spin 토글 4곳 → 0곳
  behavior_plugins에 항상 등록해두고(아무도 안 부르면 비용 0) 실제 사용은
  BT xml이 정하게 변경. yaml과 xml이 어긋나 죽는 상태가 원천 제거됨.

■ scripts/stop_all.sh
  시뮬 재시작 전 좀비 정리. 남은 ekf_local이 죽은 Gazebo의 옛 시계로
  얼어붙은 TF를 쏴서 "Gazebo는 움직이는데 RViz는 멈춤"이 발생한다.
  스크립트로 만든 이유: pkill -f를 터미널에 직접 치면 그 명령줄 자체가
  패턴에 걸려 셸이 자기를 죽인다. 또 리눅스는 프로세스 이름을 15글자까지만
  저장해 robot_state_publisher(21) 등은 pkill -x로 안 죽는다.

■ 검증 (시뮬)
  lifecycle 6개 노드 active / ERROR 0, narrow·wide 둘 다
  자율주행 목표 도달 오차 11.8~13.7 cm (허용 15), 속도 최대 정확히 0.150
  원형 순찰 12 웨이포인트 11/12 · 12/12 성공
  footprint 실측 0.218 x 0.441 m, inflation 실측 0.255 m — 설정값과 일치

Co-Authored-By: Claude Opus 5 <noreply@anthropic.com>

File: edge/ros2_ws/src/ship_ugv_description/urdf/ship_ugv_core.urdf.xacro (robot description, xacro)
@@ -88,4 +88,24 @@
     </inertial>
   </xacro:macro>
+  <!-- ================= 표시 색상 (RViz 전용) =================
+       물리·좌표와 무관하며 RViz 렌더링에만 쓰인다.
+       (Gazebo 화면 색은 ship_ugv_gazebo.xacro의 <gazebo> 태그가 따로 담당한다.
+        RViz는 <gazebo> 안을 읽지 않으므로 여기에도 정의해야 한다.)
+       색을 구분해두는 실용적 이유: RViz에서 로봇이 전부 흰색이면
+       앞뒤를 구분할 수 없다. base_link가 차체 중심이 아니라 뒷바퀴 축이라
+       "차체가 앞으로 얼마나 튀어나왔는지"를 눈으로 확인해야 할 일이 많다.
+       전방에 달린 라이다를 빨강으로 칠해 앞쪽 표식으로 쓴다. -->
+  <material name="chassis_grey">
+    <color rgba="0.25 0.27 0.30 1.0"/>
+  </material>
+  <material name="wheel_black">
+    <color rgba="0.10 0.10 0.10 1.0"/>
+  </material>
+  <material name="caster_silver">
+    <color rgba="0.70 0.70 0.72 1.0"/>
+  </material>
+  <material name="laser_red">
+    <color rgba="0.85 0.15 0.15 1.0"/>
+  </material>
   <!-- ================= base_link ================= -->
   <!-- 물리적 실체 없는 기준 프레임. 실제 차체는 chassis_link로 분리
@@ -103,4 +123,5 @@
         <box size="${chassis_length} ${chassis_width} ${chassis_height}"/>
       </geometry>
+      <material name="chassis_grey"/>
     </visual>
     <collision>
@@ -124,4 +145,5 @@
           <cylinder radius="${wheel_radius}" length="${wheel_width}"/>
         </geometry>
+        <material name="wheel_black"/>
       </visual>
       <collision>
@@ -148,4 +170,5 @@
         <sphere radius="${caster_radius}"/>
       </geometry>
+      <material name="caster_silver"/>
     </visual>
     <collision>
@@ -183,4 +206,5 @@
         <cylinder radius="0.03" length="0.04"/>
       </geometry>
+      <material name="laser_red"/>
     </visual>
     <xacro:cylinder_inertial mass="${sensor_mass}" r="0.03" h="0.04"/>
